File: Starbie.kicad_sch (KiCad schematic)
At the start: 0 parts

Commit message: Declined restore: 5 files changed fp-lib-table 4/0/0 Starbie.kicad_pcb 4274/0/0 Starbie.kicad_pro 679/0/0 Starbie.kicad_sch 2329/0/4 sym-lib-table 4/0/0
Parts:
- added J1: OLED, Starbie_Parts:Display_128x64_096_I2C, symbol Connector_Generic:Conn_01x04
- added J2: MPU6050, Starbie_Parts:MPU6050_Module, symbol Connector_Generic:Conn_01x08
- added R1: 10k, Resistor_THT:R_Axial_DIN0204_L3.6mm_D1.6mm_P7.62mm_Horizontal, symbol Device:R
- added SW1, SW2: SW_Push, Button_Switch_Keyboard:SW_Cherry_MX_1.00u_PCB, symbol Switch:SW_Push
- added U1: DHT11, Sensor:Aosong_DHT11_5.5x12.0_P2.54mm, symbol Sensor:DHT11
- added U2: XIAO-ESP32-C3-SMD, Starbie_Parts:XIAO-ESP32-C3-SMD, symbol Seeed_Studio_XIAO_Series:XIAO-ESP32-C3-SMD
Connections:
- new net +3V3: J1.2 (Pin_2), J2.1 (Pin_1), R1.1, U1.1 (VDD), U2.12 (3V3_OUT)
- new net +5V: U2.14 (VBUS)
- new net BUTTON1: SW1.1, U2.3 (D2)
- new net BUTTON2: SW2.1, U2.4 (D3)
- new net DHT11_DATA: R1.2, U1.2 (DATA), U2.2 (D1)
- new net GND: J1.1 (Pin_1), J2.2 (Pin_2), SW1.2, SW2.2, U1.4 (GND), U2.13 (GND)
- new net SCL: J1.3 (Pin_3), J2.3 (Pin_3), U2.6 (D5)
- new net SDA: J1.4 (Pin_4), J2.4 (Pin_4), U2.5 (D4)
- no-connect marks 0 -> 19
Other:
- note added: "BUTTONS"
- note added: "ENVIRONMENT SENSOR"
- note added: "ESP32-C3 (Seeed XIAO)"
- note added: "MPU6050 (GY-521)"
- note added: "OLED 128x64 (I2C)"
- note added: "POWER FLAGS"
- title: (none) -> Starbie

Commit message: Restored from 66e12344b9998c837c91bd681a67321394a8b752: 1 files changed Starbie.kicad_sch 0/2329/4
Parts:
- removed J1: OLED, Starbie_Parts:Display_128x64_096_I2C, symbol Connector_Generic:Conn_01x04
- removed J2: MPU6050, Starbie_Parts:MPU6050_Module, symbol Connector_Generic:Conn_01x08
- removed R1: 10k, Resistor_THT:R_Axial_DIN0204_L3.6mm_D1.6mm_P7.62mm_Horizontal, symbol Device:R
- removed SW1, SW2: SW_Push, Button_Switch_Keyboard:SW_Cherry_MX_1.00u_PCB, symbol Switch:SW_Push
- removed U1: DHT11, Sensor:Aosong_DHT11_5.5x12.0_P2.54mm, symbol Sensor:DHT11
- removed U2: XIAO-ESP32-C3-SMD, Starbie_Parts:XIAO-ESP32-C3-SMD, symbol Seeed_Studio_XIAO_Series:XIAO-ESP32-C3-SMD
Connections:
- no-connect marks 19 -> 0
Other:
- note removed: "BUTTONS"
- note removed: "ENVIRONMENT SENSOR"
- note removed: "ESP32-C3 (Seeed XIAO)"
- note removed: "MPU6050 (GY-521)"
- note removed: "OLED 128x64 (I2C)"
- note removed: "POWER FLAGS"
- title: Starbie -> (none)
